File: hardware/kicad/Dual_PWM_Fan_Controller/Dual_PWM_Fan_Controller.kicad_pcb (KiCad board)
At the start: 2 copper layers, 90 x 60 mm, 40 parts, among them J1 Conn_01x02, J2 Conn_01x04, J3 Conn_01x04, J4 Conn_01x02, J5 Conn_01x02, J6 Conn_01x03, J7 LED Panel, Q1 2N7002, Q2 2N7002, U1 ATtiny1616-S, U2 L78L05_SO8

Commit message: end of v0.1
Parts:
- moved J7 10.2 mm to (143.2, 67.4)
- moved R10 10.2 mm to (145.7, 76.0)
- moved R11 10.2 mm to (148.2, 76.0)
- moved R12 10.2 mm to (150.7, 76.0)
- moved R13 10.2 mm to (153.2, 76.0)
- moved R9 10.2 mm to (143.2, 76.0)
Routing:
- net Net-(U1-PA3): track 0.00 -> 30.2 mm, vias 0 -> 2
- net /LED_TH1_FAULT: track 0.00 -> 7.54 mm
- net /LED_OK: track 0.00 -> 7.54 mm
- net +5V: track 237.5 -> 238.2 mm
Changed lines of the file:
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@@
 	(footprint "Resistor_SMD:R_0805_2012Metric_Pad1.20x1.40mm_HandSolder"
 		(layer "F.Cu")
-		(at 133.025 76.5 90)
+		(at 143.187 75.962 90)
 		(descr "Resistor SMD 0805 (2012 Metric), square (rectangular) end terminal, IPC-7351 nominal with elongated pad for handsoldering. (Body size source: IPC-SM-782 page 72, https://www.pcb-3d.com/wordpress/wp-content/uploads/ipc-sm-782a_amendment_1_and_2.pdf)")
 		(tags "resistor handsolder")
@@
 	(footprint "Resistor_SMD:R_0805_2012Metric_Pad1.20x1.40mm_HandSolder"
 		(layer "F.Cu")
-		(at 143 76.5 90)
+		(at 153.162 75.962 90)
 		(descr "Resistor SMD 0805 (2012 Metric), square (rectangular) end terminal, IPC-7351 nominal with elongated pad for handsoldering. (Body size source: IPC-SM-782 page 72, https://www.pcb-3d.com/wordpress/wp-content/uploads/ipc-sm-782a_amendment_1_and_2.pdf)")
 		(tags "resistor handsolder")
@@
 	(footprint "Resistor_SMD:R_0805_2012Metric_Pad1.20x1.40mm_HandSolder"
 		(layer "F.Cu")
-		(at 135.525 76.5 90)
+		(at 145.687 75.962 90)
 		(descr "Resistor SMD 0805 (2012 Metric), square (rectangular) end terminal, IPC-7351 nominal with elongated pad for handsoldering. (Body size source: IPC-SM-782 page 72, https://www.pcb-3d.com/wordpress/wp-content/uploads/ipc-sm-782a_amendment_1_and_2.pdf)")
 		(tags "resistor handsolder")
@@
 	(footprint "Resistor_SMD:R_0805_2012Metric_Pad1.20x1.40mm_HandSolder"
 		(layer "F.Cu")
-		(at 138 76.5 90)
+		(at 148.162 75.962 90)
 		(descr "Resistor SMD 0805 (2012 Metric), square (rectangular) end terminal, IPC-7351 nominal with elongated pad for handsoldering. (Body size source: IPC-SM-782 page 72, https://www.pcb-3d.com/wordpress/wp-content/uploads/ipc-sm-782a_amendment_1_and_2.pdf)")
 		(tags "resistor handsolder")
@@
 	(footprint "Resistor_SMD:R_0805_2012Metric_Pad1.20x1.40mm_HandSolder"
 		(layer "F.Cu")
-		(at 140.5 76.5 90)
+		(at 150.662 75.962 90)
 		(descr "Resistor SMD 0805 (2012 Metric), square (rectangular) end terminal, IPC-7351 nominal with elongated pad for handsoldering. (Body size source: IPC-SM-782 page 72, https://www.pcb-3d.com/wordpress/wp-content/uploads/ipc-sm-782a_amendment_1_and_2.pdf)")
 		(tags "resistor handsolder")
@@
 	(footprint "Connector_JST:JST_XH_B6B-XH-A_1x06_P2.50mm_Vertical"
 		(layer "F.Cu")
-		(at 133 67.975)
+		(at 143.162 67.437)
 		(descr "JST XH series connector, B6B-XH-A (http://www.jst-mfg.com/product/pdf/eng/eXH.pdf)")
 		(tags "connector JST XH vertical")
@@
 	)
 	(segment
-		(start 141.12 89.88)
-		(end 140 91)
-		(width 0.5)
-		(layer "F.Cu")
-		(net "+5V")
-	)
-	(segment
 		(start 130.175 106.553)
 		(end 130.175 97.5)
@@
 	)
 	(segment
-		(start 140 96)
-		(end 138.5 97.5)
-		(width 0.5)
-		(layer "F.Cu")
-		(net "+5V")
-	)
-	(segment
 		(start 132 91.07)
 		(end 132.025 91.095)
@@
 	)
 	(segment
-		(start 140 91)
-		(end 140 96)
-		(width 0.5)
-		(layer "F.Cu")
-		(net "+5V")
-	)
-	(segment
 		(start 162.814 87.757)
 		(end 158.496 87.757)
@@
 	)
 	(segment
-		(start 138.5 97.5)
-		(end 130.175 97.5)
-		(width 0.5)
-		(layer "F.Cu")
-		(net "+5V")
-	)
-	(segment
 		(start 144.991 85.725)
 		(end 144.991 87.757)
@@
 	)
 	(segment
-		(start 141.351 89.88)
-		(end 141.12 89.88)
+		(start 145 89.88)
+		(end 140 89.88)
+		(width 0.5)
+		(layer "F.Cu")
+		(net "+5V")
+	)
+	(segment
+		(start 140 89.88)
+		(end 140 96)
 		(width 0.5)
 		(layer "F.Cu")
@@
 	)
 	(segment
-		(start 145 89.88)
-		(end 141.351 89.88)
+		(start 135.414 111.76)
+		(end 139.065 111.76)
 		(width 0.5)
 		(layer "F.Cu")
@@
 	)
 	(segment
-		(start 135.414 111.76)
-		(end 139.065 111.76)
+		(start 141.595767 84.328)
+		(end 145.034 84.328)
 		(width 0.5)
 		(layer "F.Cu")
@@
 	)
 	(segment
-		(start 141.595767 84.328)
-		(end 145.034 84.328)
+		(start 138.5 97.5)
+		(end 130.175 97.5)
 		(width 0.5)
 		(layer "F.Cu")
@@
 	)
 	(segment
+		(start 140 96)
+		(end 138.5 97.5)
+		(width 0.5)
+		(layer "F.Cu")
+		(net "+5V")
+	)
+	(segment
 		(start 128.758 79.863)
 		(end 129.54 80.645)
@@
 	)
 	(segment
+		(start 143.187 76.962)
+		(end 143.187 80.645)
+		(width 0.3)
+		(layer "F.Cu")
+		(net "Net-(U1-PA3)")
+	)
+	(segment
+		(start 156.591 88.9)
+		(end 154.686 88.9)
+		(width 0.3)
+		(layer "F.Cu")
+		(net "Net-(U1-PA3)")
+	)
+	(segment
+		(start 156.754 91.15)
+		(end 157.353 90.551)
+		(width 0.3)
+		(layer "F.Cu")
+		(net "Net-(U1-PA3)")
+	)
+	(segment
+		(start 154.432 88.646)
+		(end 154.432 88.519)
+		(width 0.3)
+		(layer "F.Cu")
+		(net "Net-(U1-PA3)")
+	)
+	(segment
+		(start 154.3 91.15)
+		(end 156.754 91.15)
+		(width 0.3)
+		(layer "F.Cu")
+		(net "Net-(U1-PA3)")
+	)
+	(segment
+		(start 157.353 90.551)
+		(end 157.353 89.662)
+		(width 0.3)
+		(layer "F.Cu")
+		(net "Net-(U1-PA3)")
+	)
+	(segment
+		(start 154.432 81.123)
+		(end 143.665 81.123)
+		(width 0.3)
+		(layer "F.Cu")
+		(net "Net-(U1-PA3)")
+	)
+	(segment
+		(start 157.353 89.662)
+		(end 156.591 88.9)
+		(width 0.3)
+		(layer "F.Cu")
+		(net "Net-(U1-PA3)")
+	)
+	(segment
+		(start 143.665 81.123)
+		(end 143.187 80.645)
+		(width 0.3)
+		(layer "F.Cu")
+		(net "Net-(U1-PA3)")
+	)
+	(segment
+		(start 154.686 88.9)
+		(end 154.432 88.646)
+		(width 0.3)
+		(layer "F.Cu")
+		(net "Net-(U1-PA3)")
+	)
+	(via
+		(at 154.432 81.123)
+		(size 0.6)
+		(drill 0.3)
+		(layers "F.Cu" "B.Cu")
+		(net "Net-(U1-PA3)")
+	)
+	(via
+		(at 154.432 88.519)
+		(size 0.6)
+		(drill 0.3)
+		(layers "F.Cu" "B.Cu")
+		(net "Net-(U1-PA3)")
+	)
+	(segment
+		(start 154.432 88.519)
+		(end 154.432 81.123)
+		(width 0.3)
+		(layer "B.Cu")
+		(net "Net-(U1-PA3)")
+	)
+	(segment
 		(start 156.718 94.996)
 		(end 156.682 94.96)
@@
 	)
 	(segment
+		(start 143.187 74.962)
+		(end 143.187 67.462)
+		(width 0.3)
+		(layer "F.Cu")
+		(net "/LED_OK")
+	)
+	(segment
+		(start 143.187 67.462)
+		(end 143.162 67.437)
+		(width 0.3)
+		(layer "F.Cu")
+		(net "/LED_OK")
+	)
+	(segment
+		(start 145.687 74.962)
+		(end 145.687 67.462)
+		(width 0.3)
+		(layer "F.Cu")
+		(net "/LED_TH1_FAULT")
+	)
+	(segment
+		(start 145.687 67.462)
+		(end 145.662 67.437)
+		(width 0.3)
+		(layer "F.Cu")
+		(net "/LED_TH1_FAULT")
+	)
+	(segment
