File: v1.0/5V/1 Fan/5V_1Fan/5V_1Fan.kicad_sch (KiCad schematic)
At the start: 19 parts, among them J1 Conn_01x03_Pin, J2 Conn_01x02, J3 Conn_01x04, J4 Conn_01x02, J5 Conn_01x03, Q1 2N7002, Q2 Q_PMOS_GSD, U1 ATtiny402-SS

Commit message: 5v 1fan 1th
Connections:
- net GREEN_LED: now also U1.3 (PA7); no longer U1.2 (PA6)
- net RED_LED: now also U1.2 (PA6); no longer U1.3 (PA7)
Changed lines of the file:
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@@
 	)
 	(label "GREEN_LED"
-		(at 113.03 95.25 0)
+		(at 113.03 97.79 0)
 		(effects
 			(font
@@
 	)
 	(label "RED_LED"
-		(at 113.03 97.79 0)
+		(at 113.03 95.25 0)
 		(effects
 			(font

Commit message: updated files
Parts:
- C1, C2: JLCPCB Part (none) -> C77082; MPN (none) -> GRM21BR71H104KA01L; Manufacturer (none) -> Murata Electronics
- C3, C4: JLCPCB Part (none) -> C380363; MPN (none) -> TCC1206X7R106K160HT; Manufacturer (none) -> CCTC
- F1: value 250mA -> 250mA PPTC; JLCPCB Part (none) -> C3762322; MPN (none) -> 1206L025/24YR; Manufacturer (none) -> Littelfuse
- J1: JLCPCB Part (none) -> C5116482; MPN (none) -> 2.54-1*3; Manufacturer (none) -> ZHOURI
- J2: JLCPCB Part (none) -> C20504437; MPN (none) -> B2B-PH-K-S; Manufacturer (none) -> JST
- J3: footprint Connector_Molex:Molex_KK-254_AE-6410-04A_1x04_P2.54mm_Vertical -> Connector:FanPinHeader_1x04_P2.54mm_Vertical; JLCPCB Part (none) -> C240840; MPN (none) -> 470531000; Manufacturer (none) -> Molex
- J4: JLCPCB Part (none) -> C158012; MPN (none) -> B2B-XH-A(LF)(SN); Manufacturer (none) -> JST
- J5: JLCPCB Part (none) -> C131339; MPN (none) -> B3B-PH-K-S(LF)(SN); Manufacturer (none) -> JST
- Q1: JLCPCB Part (none) -> C389059; MPN (none) -> 2N7002; Manufacturer (none) -> Yangzhou Yangjie Electronic Technology
- Q2: value Q_PMOS_GSD -> AO3401A; JLCPCB Part (none) -> C15127; MPN (none) -> AO3401A; Manufacturer (none) -> Alpha & Omega Semiconductor
- R1, R4: JLCPCB Part (none) -> C84376; MPN (none) -> RC0805FR-0710KL; Manufacturer (none) -> YAGEO
- R2, R5, R6: JLCPCB Part (none) -> C95781; MPN (none) -> RC0805FR-071KL; Manufacturer (none) -> YAGEO
- R3: JLCPCB Part (none) -> C96346; MPN (none) -> RC0805FR-07100KL; Manufacturer (none) -> YAGEO
- U1: value ATtiny402-SS -> ATTINY402-SSF; JLCPCB Part (none) -> C1338236; MPN (none) -> ATTINY402-SSF; Manufacturer (none) -> Microchip Technology
