File: v1.0/1 Fan 1TH/1 Fan 1 TH/1 Fan 1 TH.kicad_sch (KiCad schematic)
At the start: 51 parts, among them J1 POWER_HARNESS, J2 UPDI, J3 TH1, J4 FAN1, J5 LED_PANEL, J6 FAN2, J7 TH1, Q1 NCE40P05Y, Q2 AO3400A, Q3 AO3400A, U1 CJ7533S, U2 ATtiny1616-S

Commit message: Update 1 Fan 1 TH.kicad_sch
mosfet and mistake on th2 naming fixed
Parts:
- J7: value TH1 -> TH2
- Q1: value NCE40P05Y -> AP40P05
Changed lines of the file:
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@@
 			)
 		)
-		(property "Value" "NCE40P05Y"
+		(property "Value" "AP40P05"
 			(at 50.8 78.7399 0)
 			(show_name no)
@@
 			)
 		)
-		(property "Value" "TH1"
+		(property "Value" "TH2"
 			(at 105.41 134.6199 0)
 			(show_name no)
