File: v1.0/2 Fan 2 Th/2 Fan 2 Th.kicad_sch (KiCad schematic)
At the start: 51 parts, among them J1 POWER_HARNESS, J2 UPDI, J3 TH1, J4 FAN1, J5 LED_PANEL, J6 FAN2, J7 TH2, Q1 AP40P05, Q2 AO3400A, Q3 AO3400A, U1 CJ7533S, U2 ATtiny1616-S

Commit message: update
- pcb design started
-
Parts:
- added J8: BUZZER_HARNESS, Connector_Molex:Molex_Micro-Fit_3.0_43045-0215_2x01_P3.00mm_Vertical, symbol Connector_Generic:Conn_01x02
- added Q4: AO3400A, Package_TO_SOT_SMD:SOT-23, symbol Transistor_FET:AO3400A
- added R24: 100 Ω, Resistor_SMD:R_0603_1608Metric, symbol Device:R
- added R25: 100 kΩ, Resistor_SMD:R_0603_1608Metric, symbol Device:R
- C1: footprint (none) -> Capacitor_SMD:CP_Elec_6.3x7.7
- C10, C11, C13, C2, C3, C4, C5, C6, C7, C9: footprint (none) -> Capacitor_SMD:C_0805_2012Metric
- C12, C8: value 10 µF 35 V -> 10 µF 50 V; footprint (none) -> Capacitor_SMD:C_1210_3225Metric
- D1: footprint (none) -> Diode_SMD:D_SOD-123
- D2: footprint (none) -> Diode_SMD:D_SMB
- F1: footprint (none) -> Fuse:Fuse_1812_4532Metric
- J1, J3, J7: footprint (none) -> Connector_Molex:Molex_Micro-Fit_3.0_43045-0215_2x01_P3.00mm_Vertical
- J2: footprint (none) -> Connector_PinHeader_2.54mm:PinHeader_1x03_P2.54mm_Vertical
- J4, J6: footprint (none) -> Connector_Molex:Molex_Micro-Fit_3.0_43045-0415_2x02_P3.00mm_Vertical
- J5: footprint (none) -> Connector_Molex:Molex_Micro-Fit_3.0_43045-1015_2x05_P3.00mm_Vertical
- Q1: footprint (none) -> Package_TO_SOT_SMD:SOT-23
- R1, R10, R11, R12, R13, R14, R15, R16, R17, R18, R19, R2, R20, R21, R22, R23, R3, R4, R5, R6, R7, R8, R9: footprint (none) -> Resistor_SMD:R_0603_1608Metric
Connections:
- net FAN1_LED_A: now also J5.2 (Pin_2), R11.1; no longer J5.3 (Pin_3), R6.1
- net FAN1_LED_A_CTRL: now also R11.2; no longer R6.2
- net FAN1_LED_B: now also J5.7 (Pin_7), R14.2; no longer J5.4 (Pin_4), R7.2
- net FAN1_LED_B_CTRL: now also R14.1; no longer R7.1
- net FAN2_LED_A: now also J5.4 (Pin_4), R7.2; no longer J5.7 (Pin_7), R14.2
- net FAN2_LED_A_CTRL: now also R7.1; no longer R14.1
- net FAN2_LED_B: now also J5.9 (Pin_9), R15.2; no longer J5.8 (Pin_8), R16.1
- net FAN2_LED_B_CTRL: now also R15.1; no longer R16.2
- net GND: now also Q4.2 (S), R25.2
- net SYSTEM_LED_B: now also J5.6 (Pin_6), R9.2; no longer J5.2 (Pin_2), R11.1
- net SYSTEM_LED_B_CTRL: now also R9.1; no longer R11.2
- net TH1_LED_A: now also J5.3 (Pin_3), R6.1; no longer J5.5 (Pin_5), R8.1
- net TH1_LED_A_CTRL: now also R6.2; no longer R8.2
- net TH1_LED_B: now also J5.8 (Pin_8), R16.1; no longer J5.6 (Pin_6), R9.2
- net TH1_LED_B_CTRL: now also R16.2; no longer R9.1
- net TH2_LED_A: now also J5.5 (Pin_5), R8.1; no longer J5.9 (Pin_9), R15.2
- net TH2_LED_A_CTRL: now also R8.2; no longer R15.1
- net VIN_PROTECTED: now also J8.1 (Pin_1)
- net BUZZER_CTRL: now reaches U2.15 (PC3)
- net BUZZER_CTRL: now also R24.1
- new net: Q4.1 (G), R24.2, R25.1
- new net BUZZER_SW: J8.2 (Pin_2), Q4.3 (D)
- no-connect marks 1 -> 0
Other:
- note added: "CPE-270 1 = + 2 = –"
- moved on the sheet: C1

Commit message: design update
- silkscreen edited
- mosfet changed
- connectors type changed
- fuse changed
Parts:
- removed Q1: AP40P05, Package_TO_SOT_SMD:SOT-23, symbol Transistor_FET:Q_PMOS_GSD
- added Q1: DMPH4029LFGQ, Package_SON:Diodes_PowerDI3333-8, symbol Transistor_FET:DMP3013SFV
- F1: value 2.5A PTC -> 2920L260/24DR; footprint Fuse:Fuse_1812_4532Metric -> Fuse:Fuse_2920_7451Metric; JLCPCB (none) -> C315904; MPN (none) -> 2920L260/24DR; Manufacturer (none) -> Littelfuse
- J1, J3, J7, J8: footprint Connector_Molex:Molex_Micro-Fit_3.0_43045-0215_2x01_P3.00mm_Vertical -> Connector_Molex:Molex_Micro-Fit_3.0_43045-0218_2x01-1MP_P3.00mm_Vertical; JLCPCB (none) -> C476811; MPN (none) -> 43045-0218; Manufacturer (none) -> Molex
- J4, J6: footprint Connector_Molex:Molex_Micro-Fit_3.0_43045-0415_2x02_P3.00mm_Vertical -> Connector_Molex:Molex_Micro-Fit_3.0_43045-0418_2x02-1MP_P3.00mm_Vertical; JLCPCB (none) -> C293535; MPN (none) -> 43045-0418; Manufacturer (none) -> Molex
- J5: footprint Connector_Molex:Molex_Micro-Fit_3.0_43045-1015_2x05_P3.00mm_Vertical -> Connector_Molex:Molex_Micro-Fit_3.0_43045-1018_2x05-1MP_P3.00mm_Vertical
- U1: JLCPCB (none) -> C2829417; MPN (none) -> CJ7533S; Manufacturer (none) -> Jiangsu Changjing Electronics Technology Co., Ltd.
- U2: value ATtiny1616-S -> ATTINY1616-SNR; EEPROM (none) -> 256 B; Flash (none) -> 16 KB; JLCPCB (none) -> C609652; MPN (none) -> ATTINY1616-SNR; Manufacturer (none) -> Microchip Technology Inc.; Max clock (none) -> 20 MHz; Operating temp (none) -> -40°C to +105°C; Package (none) -> SOIC-20-300mil; SRAM (none) -> 2 KB; Supply (none) -> 1.8 V to 5.5 V
Connections:
- net VIN_FUSED: now also Q1.5 (D)
- net VIN_PROTECTED: now also Q1.1 (S), Q1.2 (S), Q1.3 (S)
- net at D1.2 (A), R1.2: now also Q1.4 (G)

Commit message: F2Th2 Finalized
F2Th2 finalized
Parts:
- C1: value 100uF 35V -> 100 µF 35V; JLCPCB (none) -> C176683; MPN (none) -> VZH101M1VTR-0607; Manufacturer (none) -> Lelon
- C10, C9: Dielectric (none) -> X7R; JLCPCB (none) -> C49678; MPN (none) -> CC0805KRX7R9BB104; Manufacturer (none) -> YAGEO; Tolerance (none) -> ±10%
- C11, C7: Dielectric (none) -> X7R; JLCPCB (none) -> C5576121; MPN (none) -> AC0805KPX7R9BB102; Manufacturer (none) -> YAGEO; Tolerance (none) -> ±10%
- C12, C8: Dielectric (none) -> X7R; JLCPCB (none) -> C5596896; MPN (none) -> CL32B106KBVZNWE; Manufacturer (none) -> Samsung Electro-Mechanics; Operating temp (none) -> -55°C to +125°C
- C13, C5, C6: value 100 nF 50V -> 100 nF 50 V; Dielectric (none) -> X7R; JLCPCB (none) -> C49678; MPN (none) -> CC0805KRX7R9BB104; Manufacturer (none) -> YAGEO; Tolerance (none) -> ±10%
- C2: value 100nF 50V -> 100 nF 50 V; Dielectric (none) -> X7R; JLCPCB (none) -> C49678; MPN (none) -> CC0805KRX7R9BB104; Manufacturer (none) -> YAGEO; Tolerance (none) -> ±10%
- C3, C4: value 1uF 50V -> 1 µF 50 V; Dielectric (none) -> X7R; JLCPCB (none) -> C28323; MPN (none) -> CL21B105KBFNNNE; Manufacturer (none) -> Samsung Electro-Mechanics; Tolerance (none) -> ±10%
- D1: JLCPCB (none) -> C173432; MPN (none) -> BZT52C8V2; Manufacturer (none) -> MDD (Microdiode Semiconductor)
- D2: JLCPCB (none) -> C78809; MPN (none) -> SMBJ15CA; Manufacturer (none) -> Littelfuse
- J2: JLCPCB (none) -> C49257; MPN (none) -> 2.54-1*3PPin; Manufacturer (none) -> BOOMELE (Boom Precision Elec); Mounting (none) -> Through Hole; Pins (none) -> 3; Pitch (none) -> 2.54 mm
- J5: JLCPCB (none) -> C476814; MPN (none) -> 43045-1018; Manufacturer (none) -> Molex
- Q1: JLCPCB (none) -> C3279395
- Q2, Q3, Q4: JLCPCB (none) -> C20917; MPN (none) -> AO3400A; Manufacturer (none) -> Alpha & Omega Semiconductor
- R1, R2, R21, R22, R5: JLCPCB (none) -> C25804; MPN (none) -> 0603WAF1002T5E; Manufacturer (none) -> UNI-ROYAL (Uniroyal Elec); Tolerance (none) -> ±1%
- R10, R11, R14, R15, R16, R17, R6, R7, R8, R9: JLCPCB (none) -> C22962; MPN (none) -> 0603WAF2200T5E; Manufacturer (none) -> UNI-ROYAL (Uniroyal Elec); Tolerance (none) -> ±1%
- R12, R13, R20, R23: JLCPCB (none) -> C21190; MPN (none) -> 0603WAF1001T5E; Manufacturer (none) -> UNI-ROYAL (Uniroyal Elec); Tolerance (none) -> ±1%
- R18, R24, R4: JLCPCB (none) -> C22775; MPN (none) -> 0603WAF1000T5E; Manufacturer (none) -> UNI-ROYAL (Uniroyal Elec); Tolerance (none) -> ±1%
- R19, R25, R3: JLCPCB (none) -> C25803; MPN (none) -> 0603WAF1003T5E; Manufacturer (none) -> UNI-ROYAL (Uniroyal Elec); Tolerance (none) -> ±1%

Commit message: simulations & silkscreen edits
Parts:
- removed Q2, Q3: AO3400A, Package_TO_SOT_SMD:SOT-23, symbol Transistor_FET:AO3400A
- added C14, C15: 10 µF 50 V, Capacitor_SMD:C_1210_3225Metric, symbol Device:C
- added C16, C17: 100 nF 50 V, Capacitor_SMD:C_0805_2012Metric, symbol Device:C
- added R26, R28: 33 Ω, Resistor_SMD:R_0603_1608Metric, symbol Device:R
- added R27: 330 Ω, Resistor_SMD:R_0805_2012Metric, symbol Device:R
- added U3: TPS7B6950QDBVRQ1, Package_TO_SOT_SMD:SOT-23-5, symbol ThermoLoop_PWM:TPS7B6950QDBVRQ1
- added U4, U5: SN74AHCT1G04DBVR, Package_TO_SOT_SMD:SOT-23-5, symbol ThermoLoop_PWM:SN74AHCT1G04DBVR
- R10, R11, R14, R15, R16, R17, R6, R7, R8, R9: value 220 Ω -> 150 Ω; JLCPCB C22962 -> C22808; MPN 0603WAF2200T5E -> 0603WAF1500T5E
Connections:
- net FAN1_PWM: now also R26.2
- net FAN2_PWM: now also R28.2
- net GND: now also C14.2, C15.2, C16.2, C17.2, R27.2, U3.3 (GND), U3.4 (GND), U4.3 (GND), U5.3 (GND)
- net VIN_PROTECTED: now also C14.1, U3.1 (IN)
- net FAN2_PWM_IN: now reaches R18.2, R19.1
- net FAN2_PWM_IN: now also U5.2 (A)
- net FAN1_PWM_IN: now reaches R3.1, R4.2
- net FAN1_PWM_IN: now also U4.2 (A)
- new net +5V_PWM: C15.1, C16.1, C17.1, R27.1, U3.5 (OUT), U4.5 (VCC), U5.5 (VCC)
- new net FAN1_PWM_DRIVE: R26.1, U4.4 (~{Y})
- new net FAN2_PWM_DRIVE: R28.1, U5.4 (~{Y})
- no-connect marks 0 -> 3
Other:
- note added: "5 V PWM DRIVER ONLY - FAN POWER REMAINS 12 V"
- note added: "Input low / MCU reset = full-speed command 25 kHz, inverted drive; R27 absorbs fan pull-up current"
