File: v1.0/1 Fan 2 Th/1 Fan 2 Th.kicad_sch (KiCad schematic)
At the start: 44 parts, among them J1 POWER_HARNESS, J2 UPDI, J3 TH1, J4 FAN1, J5 LED_PANEL, J7 TH2, J8 BUZZER_HARNESS, Q1 DMPH4029LFGQ, Q2 AO3400A, Q4 AO3400A, U1 CJ7533S, U2 ATTINY1616-SNR

Commit message: added 5v rail
added 5v rail for pwm concerns of the fans
Parts:
- removed Q2: AO3400A, Package_TO_SOT_SMD:SOT-23, symbol Transistor_FET:AO3400A
- added C14, C15: 10 µF 50 V, Capacitor_SMD:C_1210_3225Metric, symbol Device:C
- added C16: 100 nF 50 V, Capacitor_SMD:C_0805_2012Metric, symbol Device:C
- added R26: 33 Ω, Resistor_SMD:R_0603_1608Metric, symbol Device:R
- added R27: 330 Ω, Resistor_SMD:R_0805_2012Metric, symbol Device:R
- added U3: TPS7B6950QDBVRQ1, Package_TO_SOT_SMD:SOT-23-5, symbol ThermoLoop_PWM:TPS7B6950QDBVRQ1
- added U4: SN74AHCT1G04DBVR, Package_TO_SOT_SMD:SOT-23-5, symbol ThermoLoop_PWM:SN74AHCT1G04DBVR
Connections:
- net FAN1_PWM: now also R26.2
- net GND: now also C14.2, C15.2, C16.2, R27.2, U3.3 (GND), U3.4 (GND), U4.3 (GND)
- net VIN_PROTECTED: now also C14.1, U3.1 (IN)
- net FAN1_PWM_IN: now reaches R3.1, R4.2
- net FAN1_PWM_IN: now also U4.2 (A)
- new net +5V_PWM: C15.1, C16.1, R27.1, U3.5 (OUT), U4.5 (VCC)
- new net FAN1_PWM_DRIVE: R26.1, U4.4 (~{Y})
- no-connect marks 6 -> 8
Other:
- note added: "5 V PWM DRIVER ONLY - FAN POWER REMAINS 12 V"
- note added: "Input low / MCU reset = full-speed command 25 kHz, inverted drive; R27 absorbs fan pull-up current"

Commit message: simulations & silkscreen edits
Parts:
- R10, R11, R14, R16, R17, R6, R8, R9: value 220 Ω -> 150 Ω; JLCPCB C22962 -> C22808; MPN 0603WAF2200T5E -> 0603WAF1500T5E
Changed lines of the file:
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@@
 			)
 		)
-		(property "Value" "220 Ω"
+		(property "Value" "150 Ω"
 			(at 71.374 174.244 90)
 			(show_name no)
@@
 			)
 		)
-		(property "Description" "220Ω ±1%, 100mW Thick Film Resistor, 0603"
+		(property "Description" "150Ω ±1%, 100mW Thick Film Resistor, 0603"
 			(at 64.77 175.26 0)
 			(hide yes)
@@
 			)
 		)
-		(property "MPN" "0603WAF2200T5E"
+		(property "MPN" "0603WAF1500T5E"
 			(at 64.77 175.26 90)
 			(hide yes)
@@
 			)
 		)
-		(property "JLCPCB" "C22962"
+		(property "JLCPCB" "C22808"
 			(at 64.77 175.26 90)
 			(hide yes)
@@
 			)
 		)
-		(property "Value" "220 Ω"
+		(property "Value" "150 Ω"
 			(at 71.374 171.704 90)
 			(show_name no)
@@
 			)
 		)
-		(property "Description" "220Ω ±1%, 100mW Thick Film Resistor, 0603"
+		(property "Description" "150Ω ±1%, 100mW Thick Film Resistor, 0603"
 			(at 64.77 172.72 0)
 			(hide yes)
@@
 			)
 		)
-		(property "MPN" "0603WAF2200T5E"
+		(property "MPN" "0603WAF1500T5E"
 			(at 64.77 172.72 90)
 			(hide yes)
@@
 			)
 		)
-		(property "JLCPCB" "C22962"
+		(property "JLCPCB" "C22808"
 			(at 64.77 172.72 90)
 			(hide yes)
@@
 			)
 		)
-		(property "Value" "220 Ω"
+		(property "Value" "150 Ω"
 			(at 121.158 179.324 90)
 			(show_name no)
@@
 			)
 		)
-		(property "Description" "220Ω ±1%, 100mW Thick Film Resistor, 0603"
+		(property "Description" "150Ω ±1%, 100mW Thick Film Resistor, 0603"
 			(at 127 180.34 0)
 			(hide yes)
@@
 			)
 		)
-		(property "MPN" "0603WAF2200T5E"
+		(property "MPN" "0603WAF1500T5E"
 			(at 127 180.34 90)
 			(hide yes)
@@
 			)
 		)
-		(property "JLCPCB" "C22962"
+		(property "JLCPCB" "C22808"
 			(at 127 180.34 90)
 			(hide yes)
@@
 			)
 		)
-		(property "Value" "220 Ω"
+		(property "Value" "150 Ω"
 			(at 71.374 179.324 90)
 			(show_name no)
@@
 			)
 		)
-		(property "Description" "220Ω ±1%, 100mW Thick Film Resistor, 0603"
+		(property "Description" "150Ω ±1%, 100mW Thick Film Resistor, 0603"
 			(at 64.77 180.34 0)
 			(hide yes)
@@
 			)
 		)
-		(property "MPN" "0603WAF2200T5E"
+		(property "MPN" "0603WAF1500T5E"
 			(at 64.77 180.34 90)
 			(hide yes)
@@
 			)
 		)
-		(property "JLCPCB" "C22962"
+		(property "JLCPCB" "C22808"
 			(at 64.77 180.34 90)
 			(hide yes)
@@
 			)
 		)
-		(property "Value" "220 Ω"
+		(property "Value" "150 Ω"
 			(at 121.158 176.784 90)
 			(show_name no)
@@
 			)
 		)
-		(property "Description" "220Ω ±1%, 100mW Thick Film Resistor, 0603"
+		(property "Description" "150Ω ±1%, 100mW Thick Film Resistor, 0603"
 			(at 127 177.8 0)
 			(hide yes)
@@
 			)
 		)
-		(property "MPN" "0603WAF2200T5E"
+		(property "MPN" "0603WAF1500T5E"
 			(at 127 177.8 90)
 			(hide yes)
@@
 			)
 		)
-		(property "JLCPCB" "C22962"
+		(property "JLCPCB" "C22808"
 			(at 127 177.8 90)
 			(hide yes)
@@
 			)
 		)
-		(property "Value" "220 Ω"
+		(property "Value" "150 Ω"
 			(at 121.158 171.704 90)
 			(show_name no)
@@
 			)
 		)
-		(property "Description" "220Ω ±1%, 100mW Thick Film Resistor, 0603"
+		(property "Description" "150Ω ±1%, 100mW Thick Film Resistor, 0603"
 			(at 127 172.72 0)
 			(hide yes)
@@
 			)
 		)
-		(property "MPN" "0603WAF2200T5E"
+		(property "MPN" "0603WAF1500T5E"
 			(at 127 172.72 90)
 			(hide yes)
@@
 			)
 		)
-		(property "JLCPCB" "C22962"
+		(property "JLCPCB" "C22808"
 			(at 127 172.72 90)
 			(hide yes)
@@
 			)
 		)
-		(property "Value" "220 Ω"
+		(property "Value" "150 Ω"
 			(at 71.374 176.784 90)
 			(show_name no)
@@
 			)
 		)
-		(property "Description" "220Ω ±1%, 100mW Thick Film Resistor, 0603"
+		(property "Description" "150Ω ±1%, 100mW Thick Film Resistor, 0603"
 			(at 64.77 177.8 0)
 			(hide yes)
@@
 			)
 		)
-		(property "MPN" "0603WAF2200T5E"
+		(property "MPN" "0603WAF1500T5E"
 			(at 64.77 177.8 90)
 			(hide yes)
@@
 			)
 		)
-		(property "JLCPCB" "C22962"
+		(property "JLCPCB" "C22808"
 			(at 64.77 177.8 90)
 			(hide yes)
@@
 			)
 		)
-		(property "Value" "220 Ω"
+		(property "Value" "150 Ω"
 			(at 121.158 181.864 90)
 			(show_name no)
@@
 			)
 		)
-		(property "Description" "220Ω ±1%, 100mW Thick Film Resistor, 0603"
+		(property "Description" "150Ω ±1%, 100mW Thick Film Resistor, 0603"
 			(at 127 182.88 0)
 			(hide yes)
@@
 			)
 		)
-		(property "MPN" "0603WAF2200T5E"
+		(property "MPN" "0603WAF1500T5E"
 			(at 127 182.88 90)
 			(hide yes)
@@
 			)
 		)
-		(property "JLCPCB" "C22962"
+		(property "JLCPCB" "C22808"
 			(at 127 182.88 90)
 			(hide yes)

Commit message: Getting Manufacturing Ready
- files updated and ordered through jlcpcb
Parts:
- C14, C15, C8: JLCPCB C5596896 -> C138687; MPN CL32B106KBVZNWE -> CL32B106KBJNNNE
- C7: JLCPCB C5576121 -> C46653; MPN AC0805KPX7R9BB102 -> CL21B102KBCNNNC; Manufacturer YAGEO -> Samsung Electro-Mechanics
Changed lines of the file:
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@@
 			)
 		)
-		(property "MPN" "CL32B106KBVZNWE"
+		(property "MPN" "CL32B106KBJNNNE"
 			(at 252.73 123.19 0)
 			(hide yes)
@@
 			)
 		)
-		(property "JLCPCB" "C5596896"
+		(property "JLCPCB" "C138687"
 			(at 252.73 123.19 0)
 			(hide yes)
@@
 			)
 		)
-		(property "Manufacturer" "YAGEO"
+		(property "Manufacturer" "Samsung Electro-Mechanics"
 			(at 247.65 142.24 0)
 			(hide yes)
@@
 			)
 		)
-		(property "MPN" "AC0805KPX7R9BB102"
+		(property "MPN" "CL21B102KBCNNNC"
 			(at 247.65 142.24 0)
 			(hide yes)
@@
 			)
 		)
-		(property "JLCPCB" "C5576121"
+		(property "JLCPCB" "C46653"
 			(at 247.65 142.24 0)
 			(hide yes)
@@
 (symbol (lib_id "ThermoLoop_PWM:TPS7B6950QDBVRQ1") (at 220.98 27.94 0) (unit 1) (in_bom yes) (on_board yes) (dnp no) (property "Reference" "U3" (at 220.98 18 0) (effects (font (size 1.0 1.0))))(property "Value" "TPS7B6950QDBVRQ1" (at 220.98 20.5 0) (effects (font (size 1.0 1.0))))(property "Footprint" "Package_TO_SOT_SMD:SOT-23-5" (at 220.98 27.94 0) (effects (font (size 1.0 1.0)) (hide yes)))(property "Datasheet" "https://www.ti.com/lit/ds/symlink/tps7b69-q1.pdf" (at 220.98 27.94 0) (effects (font (size 1.0 1.0)) (hide yes)))(property "JLCPCB" "C132202" (at 220.98 27.94 0) (effects (font (size 1.0 1.0)) (hide yes)))(property "MPN" "TPS7B6950QDBVRQ1" (at 220.98 27.94 0) (effects (font (size 1.0 1.0)) (hide yes)))(property "Manufacturer" "Texas Instruments" (at 220.98 27.94 0) (effects (font (size 1.0 1.0)) (hide yes)))(property "Description" "5 V 150 mA LDO, 40 V input, SOT-23-5" (at 220.98 27.94 0) (effects (font (size 1.0 1.0)) (hide yes)))
  (instances (project "1 Fan 2 Th" (path "/70fc5203-ff69-4e9b-b309-3a914fb06dc3" (reference "U3") (unit 1)))))
-(symbol (lib_id "Device:C") (at 203.2 35.56 0) (unit 1) (in_bom yes) (on_board yes) (dnp no) (property "Reference" "C14" (at 207.2 34.06 0) (effects (font (size 1.0 1.0))))(property "Value" "10 µF 50 V" (at 210.2 37.06 0) (effects (font (size 1.0 1.0))))(property "Footprint" "Capacitor_SMD:C_1210_3225Metric" (at 203.2 35.56 0) (effects (font (size 1.0 1.0)) (hide yes)))(property "Datasheet" "" (at 203.2 35.56 0) (effects (font (size 1.0 1.0)) (hide yes)))(property "Description" "10uF ±10%, 50V X7R MLCC, 1210" (at 203.2 35.56 0) (effects (font (size 1.0 1.0)) (hide yes)))(property "Manufacturer" "Samsung Electro-Mechanics" (at 203.2 35.56 0) (effects (font (size 1.0 1.0)) (hide yes)))(property "MPN" "CL32B106KBVZNWE" (at 203.2 35.56 0) (effects (font (size 1.0 1.0)) (hide yes)))(property "JLCPCB" "C5596896" (at 203.2 35.56 0) (effects (font (size 1.0 1.0)) (hide yes)))(property "Dielectric" "X7R" (at 203.2 35.56 0) (effects (font (size 1.0 1.0)) (hide yes)))(property "Operating temp" "-55°C to +125°C" (at 203.2 35.56 0) (effects (font (size 1.0 1.0)) (hide yes)))
+(symbol (lib_id "Device:C") (at 203.2 35.56 0) (unit 1) (in_bom yes) (on_board yes) (dnp no) (property "Reference" "C14" (at 207.2 34.06 0) (effects (font (size 1.0 1.0))))(property "Value" "10 µF 50 V" (at 210.2 37.06 0) (effects (font (size 1.0 1.0))))(property "Footprint" "Capacitor_SMD:C_1210_3225Metric" (at 203.2 35.56 0) (effects (font (size 1.0 1.0)) (hide yes)))(property "Datasheet" "" (at 203.2 35.56 0) (effects (font (size 1.0 1.0)) (hide yes)))(property "Description" "10uF ±10%, 50V X7R MLCC, 1210" (at 203.2 35.56 0) (effects (font (size 1.0 1.0)) (hide yes)))(property "Manufacturer" "Samsung Electro-Mechanics" (at 203.2 35.56 0) (effects (font (size 1.0 1.0)) (hide yes)))(property "MPN" "CL32B106KBJNNNE" (at 203.2 35.56 0) (effects (font (size 1.0 1.0)) (hide yes)))(property "JLCPCB" "C138687" (at 203.2 35.56 0) (effects (font (size 1.0 1.0)) (hide yes)))(property "Dielectric" "X7R" (at 203.2 35.56 0) (effects (font (size 1.0 1.0)) (hide yes)))(property "Operating temp" "-55°C to +125°C" (at 203.2 35.56 0) (effects (font (size 1.0 1.0)) (hide yes)))
  (instances (project "1 Fan 2 Th" (path "/70fc5203-ff69-4e9b-b309-3a914fb06dc3" (reference "C14") (unit 1)))))
-(symbol (lib_id "Device:C") (at 241.3 35.56 0) (unit 1) (in_bom yes) (on_board yes) (dnp no) (property "Reference" "C15" (at 245.3 34.06 0) (effects (font (size 1.0 1.0))))(property "Value" "10 µF 50 V" (at 248.3 37.06 0) (effects (font (size 1.0 1.0))))(property "Footprint" "Capacitor_SMD:C_1210_3225Metric" (at 241.3 35.56 0) (effects (font (size 1.0 1.0)) (hide yes)))(property "Datasheet" "" (at 241.3 35.56 0) (effects (font (size 1.0 1.0)) (hide yes)))(property "Description" "10uF ±10%, 50V X7R MLCC, 1210" (at 241.3 35.56 0) (effects (font (size 1.0 1.0)) (hide yes)))(property "Manufacturer" "Samsung Electro-Mechanics" (at 241.3 35.56 0) (effects (font (size 1.0 1.0)) (hide yes)))(property "MPN" "CL32B106KBVZNWE" (at 241.3 35.56 0) (effects (font (size 1.0 1.0)) (hide yes)))(property "JLCPCB" "C5596896" (at 241.3 35.56 0) (effects (font (size 1.0 1.0)) (hide yes)))(property "Dielectric" "X7R" (at 241.3 35.56 0) (effects (font (size 1.0 1.0)) (hide yes)))(property "Operating temp" "-55°C to +125°C" (at 241.3 35.56 0) (effects (font (size 1.0 1.0)) (hide yes)))
+(symbol (lib_id "Device:C") (at 241.3 35.56 0) (unit 1) (in_bom yes) (on_board yes) (dnp no) (property "Reference" "C15" (at 245.3 34.06 0) (effects (font (size 1.0 1.0))))(property "Value" "10 µF 50 V" (at 248.3 37.06 0) (effects (font (size 1.0 1.0))))(property "Footprint" "Capacitor_SMD:C_1210_3225Metric" (at 241.3 35.56 0) (effects (font (size 1.0 1.0)) (hide yes)))(property "Datasheet" "" (at 241.3 35.56 0) (effects (font (size 1.0 1.0)) (hide yes)))(property "Description" "10uF ±10%, 50V X7R MLCC, 1210" (at 241.3 35.56 0) (effects (font (size 1.0 1.0)) (hide yes)))(property "Manufacturer" "Samsung Electro-Mechanics" (at 241.3 35.56 0) (effects (font (size 1.0 1.0)) (hide yes)))(property "MPN" "CL32B106KBJNNNE" (at 241.3 35.56 0) (effects (font (size 1.0 1.0)) (hide yes)))(property "JLCPCB" "C138687" (at 241.3 35.56 0) (effects (font (size 1.0 1.0)) (hide yes)))(property "Dielectric" "X7R" (at 241.3 35.56 0) (effects (font (size 1.0 1.0)) (hide yes)))(property "Operating temp" "-55°C to +125°C" (at 241.3 35.56 0) (effects (font (size 1.0 1.0)) (hide yes)))
  (instances (project "1 Fan 2 Th" (path "/70fc5203-ff69-4e9b-b309-3a914fb06dc3" (reference "C15") (unit 1)))))
 (symbol (lib_id "Device:R") (at 265.43 35.56 0) (unit 1) (in_bom yes) (on_board yes) (dnp no) (property "Reference" "R27" (at 269.43 34.06 0) (effects (font (size 1.0 1.0))))(property "Value" "330 Ω" (at 272.43 37.06 0) (effects (font (size 1.0 1.0))))(property "Footprint" "Resistor_SMD:R_0805_2012Metric" (at 265.43 35.56 0) (effects (font (size 1.0 1.0)) (hide yes)))(property "Datasheet" "" (at 265.43 35.56 0) (effects (font (size 1.0 1.0)) (hide yes)))(property "Description" "330 ohm 1% 125mW 0805; shared 1/2 fan 5V minimum load / pull-up bleed" (at 265.43 35.56 0) (effects (font (size 1.0 1.0)) (hide yes)))(property "Manufacturer" "UNI-ROYAL (Uniroyal Elec)" (at 265.43 35.56 0) (effects (font (size 1.0 1.0)) (hide yes)))(property "MPN" "0805W8F3300T5E" (at 265.43 35.56 0) (effects (font (size 1.0 1.0)) (hide yes)))(property "JLCPCB" "C17630" (at 265.43 35.56 0) (effects (font (size 1.0 1.0)) (hide yes)))(property "Tolerance" "±1%" (at 265.43 35.56 0) (effects (font (size 1.0 1.0)) (hide yes)))
