File: v1.0/1 Fan 2 Th/_restore_backup_2026-09-18T16-37-54-304/1 Fan 2 Th.kicad_pcb (KiCad board)
At the start: 2 copper layers, 90 x 75 mm, 54 parts, among them J1 POWER_HARNESS, J2 UPDI, J3 TH1, J4 FAN1, J5 LED_PANEL, J7 TH2, J8 BUZZER_HARNESS, Q1 DMPH4029LFGQ, Q4 AO3400A, U1 CJ7533S, U2 ATTINY1616-SNR, U3 TPS7B6950QDBVRQ1, U4 SN74AHCT1G04DBVR

Commit message: manufacturing & enclosure design
Changed lines of the file:
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@@
 			)
 		)
-		(property "MPN" "CL32B106KBVZNWE"
+		(property "MPN" "CL32B106KBJNNNE"
 			(at 0 0 180)
 			(layer "F.SilkS")
@@
 			)
 		)
-		(property "JLCPCB" "C5596896"
+		(property "JLCPCB" "C138687"
 			(at 0 0 180)
 			(layer "F.SilkS")
@@
 			)
 		)
-		(property "MPN" "CL32B106KBVZNWE"
+		(property "MPN" "CL32B106KBJNNNE"
 			(at 0 0 0)
 			(unlocked yes)
@@
 			)
 		)
-		(property "JLCPCB" "C5596896"
+		(property "JLCPCB" "C138687"
 			(at 0 0 0)
 			(unlocked yes)
@@
 			)
 		)
-		(property "MPN" "CL32B106KBVZNWE"
+		(property "MPN" "CL32B106KBJNNNE"
 			(at 0 0 0)
 			(layer "F.SilkS")
@@
 			)
 		)
-		(property "JLCPCB" "C5596896"
+		(property "JLCPCB" "C138687"
 			(at 0 0 0)
 			(layer "F.SilkS")
@@
 			)
 		)
-		(property "Manufacturer" "YAGEO"
+		(property "Manufacturer" "Samsung Electro-Mechanics"
 			(at 0 0 90)
 			(unlocked yes)
@@
 			)
 		)
-		(property "MPN" "AC0805KPX7R9BB102"
+		(property "MPN" "CL21B102KBCNNNC"
 			(at 0 0 90)
 			(unlocked yes)
@@
 			)
 		)
-		(property "JLCPCB" "C5576121"
+		(property "JLCPCB" "C46653"
 			(at 0 0 90)
 			(unlocked yes)
@@
 	)
 	(gr_text "PROG"
-		(at 73.2 60.6 0)
+		(at 74.2 60.6 0)
 		(layer "F.SilkS")
 		(effects
@@
 	)
 	(gr_text "1 FAN•2 TH"
-		(at 91.6 101 0)
+		(at 91.6 100.9 0)
 		(layer "F.SilkS")
 		(effects
@@
 	)
 	(gr_text "v1.0  09-2026"
-		(at 91.6 102.9 0)
+		(at 91.6 102.6 0)
 		(layer "F.SilkS")
 		(effects
