File: v1.0/1 Fan 2 Th/_restore_backup_2026-09-18T16-37-54-304/1 Fan 2 Th.kicad_sch (KiCad schematic)
At the start: 50 parts, among them J1 POWER_HARNESS, J2 UPDI, J3 TH1, J4 FAN1, J5 LED_PANEL, J7 TH2, J8 BUZZER_HARNESS, Q1 DMPH4029LFGQ, Q4 AO3400A, U1 CJ7533S, U2 ATTINY1616-SNR, U3 TPS7B6950QDBVRQ1, U4 SN74AHCT1G04DBVR

Commit message: manufacturing & enclosure design
Parts:
- C14, C15, C8: JLCPCB C5596896 -> C138687; MPN CL32B106KBVZNWE -> CL32B106KBJNNNE
- C7: JLCPCB C5576121 -> C46653; MPN AC0805KPX7R9BB102 -> CL21B102KBCNNNC; Manufacturer YAGEO -> Samsung Electro-Mechanics
